File: pcb/lamp_refurb.kicad_pcb (KiCad board)
At the start: 2 copper layers, 93.8 x 23.9 mm, 13 parts, among them J1 Conn_02x05_Odd_Even, J2 Screw_Terminal_01x03, J3 Screw_Terminal_01x06, Q1 PBSS4350SS, U1 ESP32-WROOM-32D, U3 R-78E3.3-1.0

Commit message: PCB v1.1
Parts:
- added R3: 10KΩ, Resistor_SMD:R_0805_2012Metric, F.Cu at (152.4, 97.2)
- added svg2mod: G***, svg2mod, F.Cu at (106.8, 118.0)
- moved R1 1.75 mm to (84.8, 102.7)
Connections:
- U1 pad 3: (no net) -> Net-(R3-Pad1)
Routing:
- net /3.3V: track 88.0 -> 92.4 mm
- net Net-(R3-Pad1): track 0.00 -> 2.74 mm
- net /level1: track 68.3 -> 70.0 mm
- net /warm: track 30.5 -> 32.0 mm
Other:
- board text removed: "October 2020"
