File: pcb/lamp_refurb.kicad_sch (KiCad schematic)
At the start: 13 parts, among them J1 Conn_02x05_Odd_Even, J2 Screw_Terminal_01x03, J3 Screw_Terminal_01x06, Q1 PBSS4350SS, U1 ESP32-WROOM-32D, U3 R-78E3.3-1.0

Commit message: PCB v1.1
Parts:
- added R3: 10KΩ, Resistor_SMD:R_0805_2012Metric, symbol Device:R_US
Connections:
- net 3.3V: now also R3.2
- net at U1.3 (EN): now also R3.1
Other:
- moved on the sheet: C1, D1, J1, J2, J3, Q1A, Q1B, R1, R2, R4, RV1, RV2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
